File: V2.sch (KiCad schematic (older format))
At the start: 76 parts, among them J20 Boot0, J21 Bed Temp, J22 Boot1, J26 USB_A, J27 LCD, J3 Bed Heater, J31 Bed level, J32 USB_B, J6 Head2, J7 Head1, M3 Motor Z2, M4 Motor Z1, M5 Motor Y, M6 Motor X, Q1 STN4NF20L, Q2 STN4NF20L, Q3 04N03LA, Q4 04N03LA, Q5 04N03LA, Q6 04N03LA, SW10 Button DOWN, SW11 Button UP, SW2 Boundary X, SW3 Boundary Y, SW4 Boundary Z1, SW5 Boundary Z2, SW6 Boundary E1, SW7 Boundary E2, SW8 Button BACK, SW9 Button OK, U1 LM2596S-5, U2 R-783.3-1.0, U3 STM32F105VCT6, U4 CP2104, Y1 hc49s

Commit message: Драйвера перенесены вбок, новая распиновка
Parts:
- removed C7, C9: 33uF, Capacitor_SMD:CP_Elec_6.3x5.4, symbol V2-rescue:CP-device
- added J1: Input voltage, TerminalBlock_4Ucon:TerminalBlock_4Ucon_1x02_P3.50mm_Horizontal, symbol Connector:Conn_01x02
- J32: footprint Connector_USB:USB_B_Amphenol_MUSB-D511_Vertical_Rugged -> Connector_USB:USB_B_OST_USB-B1HSxx_Horizontal
- M3, M4, M5, M6: footprint Connector_JST:JST_EH_S04B-EH_1x04_P2.50mm_Horizontal -> Connector_JST:JST_EH_B04B-EH-A_1x04_P2.50mm_Vertical
- SW10, SW11, SW8, SW9: footprint Connector_PinHeader_2.54mm:PinHeader_1x02_P2.54mm_Vertical -> Button_Switch_THT:SW_PUSH_6mm
- renumbered 33uH1 to 47uH1
Connections:
- net +24V: now also J1.2 (Pin_2)
- net GND: now also J1.1 (Pin_1)
- net GNDD: now also J6.4 (Pin_4), J7.4 (Pin_4); no longer J6.8 (Pin_8), J7.8 (Pin_8)
- net at Q5.1 (G), R5.2: now also U3.30 (ADC1_IN5/ADC2_IN5/DAC_OUT2/SPI1_SCK/PA5); no longer U3.1 (PE2/SYS_TRACECLK)
- net at U3.15 (ADC1_IN10/ADC2_IN10/PC0): now also J21.1 (Pin_1), R10.1
- net at U3.16 (ADC1_IN11/ADC2_IN11/PC1): now also J31.2 (Pin_2)
- net at U3.17 (ADC1_IN12/ADC2_IN12/PC2): now also SW2.1 (A)
- net at U3.18 (ADC1_IN13/ADC2_IN13/PC3): now also SW3.1 (A)
- net at U3.23 (ADC1_IN0/ADC2_IN0/SYS_WKUP/TIM2_CH1/TIM2_ETR/TIM5_CH1/USART2_CTS/PA0): now also SW4.1 (A)
- net at U3.24 (ADC1_IN1/ADC2_IN1/TIM2_CH2/TIM5_CH2/USART2_RTS/PA1): now also SW5.1 (A)
- net at U3.26 (ADC1_IN3/ADC2_IN3/TIM2_CH4/TIM5_CH4/USART2_RX/PA3): now also SW7.1 (A); no longer J31.2 (Pin_2)
- net at U3.29 (ADC1_IN4/ADC2_IN4/DAC_OUT1/I2S3_WS/SPI1_NSS/SPI3_NSS/USART2_CK/PA4): now also J6.2 (Pin_2), R9.1; no longer SW2.1 (A)
- net at U3.31 (ADC1_IN6/ADC2_IN6/SPI1_MISO/TIM1_BKIN/TIM3_CH1/PA6): now also Q1.1 (G), R1.2; no longer SW4.1 (A)
- net at U3.32 (ADC1_IN7/ADC2_IN7/SPI1_MOSI/TIM1_CH1N/TIM3_CH2/PA7): now also A1.9 (~ENABLE); no longer SW5.1 (A)
- net at SW6.1 (A): now also U3.25 (ADC1_IN2/ADC2_IN2/TIM2_CH3/TIM5_CH3/USART2_TX/PA2); no longer U3.33 (ADC1_IN14/ADC2_IN14/PC4)
- net at U3.34 (ADC1_IN15/ADC2_IN15/PC5): now also A1.16 (DIR); no longer SW7.1 (A)
- net at R8.1, U3.35 (ADC1_IN8/ADC2_IN8/TIM1_CH2N/TIM3_CH3/PB0): now also J7.2 (Pin_2); no longer J7.6 (Pin_6)
- net at J22.2 (Pin_2), U3.37 (BOOT1/PB2): now also Q2.1 (G), R2.2
- net at U3.38 (PE7/TIM1_ETR): now also A2.9 (~ENABLE)
- net at U3.39 (PE8/TIM1_CH1N): now also A2.15 (STEP)
- net at U3.40 (PE9/DAC_EXTI9/TIM1_CH1): now also A2.16 (DIR)
- net at U3.41 (PE10/TIM1_CH2N): now also A3.9 (~ENABLE)
- net at U3.42 (PE11/ADC1_EXTI11/ADC2_EXTI11/TIM1_CH2): now also A3.15 (STEP)
- net at U3.43 (PE12/TIM1_CH3N): now also A3.16 (DIR)
- net at U3.44 (PE13/TIM1_CH3): now also A4.9 (~ENABLE)
- net at U3.45 (PE14/TIM1_CH4): now also A4.15 (STEP)
- net at U3.46 (PE15/ADC1_EXTI15/ADC2_EXTI15/TIM1_BKIN): now also A4.16 (DIR)
- net at U3.47 (I2C2_SCL/TIM2_CH3/USART3_TX/PB10): now also A5.9 (~ENABLE)
- net at U3.48 (ADC1_EXTI11/ADC2_EXTI11/I2C2_SDA/TIM2_CH4/USART3_RX/PB11): now also A5.15 (STEP)
- net at U3.51 (CAN2_RX/I2C2_SMBA/I2S2_WS/SPI2_NSS/TIM1_BKIN/USART3_CK/PB12): now also A5.16 (DIR); no longer J27.4 (Pin_4)
- net at U3.52 (CAN2_TX/I2S2_CK/SPI2_SCK/TIM1_CH1N/USART3_CTS/PB13): now also A6.16 (DIR); no longer J27.5 (Pin_5)
- net at U3.53 (SPI2_MISO/TIM1_CH2N/USART3_RTS/PB14): now also A6.15 (STEP); no longer J27.6 (Pin_6)
- net at U3.54 (ADC1_EXTI15/ADC2_EXTI15/I2S2_SD/SPI2_MOSI/TIM1_CH3N/PB15): now also A6.9 (~ENABLE); no longer J27.7 (Pin_7)
- net at U3.55 (PD8/USART3_TX): no longer J27.8 (Pin_8)
- net at U3.56 (PD9/DAC_EXTI9/USART3_RX): now also J27.4 (Pin_4); no longer J27.9 (Pin_9)
- net at U3.57 (PD10/USART3_CK): now also J27.5 (Pin_5); no longer J27.10 (Pin_10)
- net at U3.58 (PD11/ADC1_EXTI11/ADC2_EXTI11/USART3_CTS): now also J27.6 (Pin_6); no longer J27.11 (Pin_11)
- net at U3.59 (PD12/TIM4_CH1/USART3_RTS): now also J27.7 (Pin_7); no longer J27.12 (Pin_12)
- net at U3.60 (PD13/TIM4_CH2): now also J27.8 (Pin_8); no longer J27.13 (Pin_13)
- net at U3.61 (PD14/TIM4_CH3): now also J27.9 (Pin_9); no longer J27.14 (Pin_14)
- net at U3.62 (PD15/ADC1_EXTI15/ADC2_EXTI15/TIM4_CH4): now also J27.10 (Pin_10); no longer LS1.1
- net at U3.63 (I2S2_MCK/TIM3_CH1/PC6): now also J27.11 (Pin_11); no longer SW11.1
- net at U3.64 (I2S3_MCK/TIM3_CH2/PC7): now also J27.12 (Pin_12); no longer SW10.1
- net at U3.65 (TIM3_CH3/PC8): now also J27.13 (Pin_13); no longer SW9.1
- net at U3.66 (DAC_EXTI9/TIM3_CH4/PC9): now also J27.14 (Pin_14); no longer SW8.1
- net at U3.67 (RCC_MCO/TIM1_CH1/USART1_CK/USB_OTG_FS_SOF/PA8): now also Q6.1 (G), R11.2; no longer D4.2 (A)
- net at U3.7 (RTC_OUT/RTC_TAMPER/PC13): no longer A1.9 (~ENABLE)
- net at U3.76 (SYS_JTCK-SWCLK/PA14): no longer A6.16 (DIR)
- net at U3.77 (ADC1_EXTI15/ADC2_EXTI15/I2S3_WS/SPI1_NSS/SPI3_NSS/SYS_JTDI/TIM2_CH1/TIM2_ETR/PA15): no longer A6.15 (STEP)
- net at U3.78 (I2S3_CK/SPI3_SCK/UART4_TX/USART3_TX/PC10): no longer A6.9 (~ENABLE)
- net at U3.79 (ADC1_EXTI11/ADC2_EXTI11/SPI3_MISO/UART4_RX/USART3_RX/PC11): no longer A5.16 (DIR)
- net at A1.15 (STEP): now also U3.33 (ADC1_IN14/ADC2_IN14/PC4); no longer U3.8 (RCC_OSC32_IN/PC14)
- net at U3.80 (I2S3_SD/SPI3_MOSI/UART5_TX/USART3_CK/PC12): no longer A5.15 (STEP)
- net at U3.81 (PD0/CAN1_RX): no longer A5.9 (~ENABLE)
- net at U3.82 (PD1/CAN1_TX): no longer A4.16 (DIR)
- net at U3.83 (PD2/TIM3_ETR/UART5_RX): no longer A4.15 (STEP)
- net at U3.84 (PD3/USART2_CTS): no longer A4.9 (~ENABLE)
- net at U3.85 (PD4/USART2_RTS): no longer A3.16 (DIR)
- net at U3.86 (PD5/USART2_TX): no longer A3.15 (STEP)
- net at U3.87 (PD6/USART2_RX): now also D4.2 (A); no longer A3.9 (~ENABLE)
- net at U3.88 (PD7/USART2_CK): now also SW10.1; no longer A2.16 (DIR)
- net at U3.89 (I2S3_CK/SPI1_SCK/SPI3_SCK/SYS_JTDO/SYS_TRACESWO/TIM2_CH2/PB3): now also SW11.1; no longer A2.15 (STEP)
- net at U3.90 (SPI1_MISO/SPI3_MISO/SYS_NJTRST/TIM3_CH1/PB4): now also SW9.1; no longer A2.9 (~ENABLE)
- net at U3.91 (CAN2_RX/I2C1_SMBA/I2S3_SD/SPI1_MOSI/SPI3_MOSI/TIM3_CH2/PB5): now also SW8.1; no longer A1.16 (DIR)
- net at Q4.1 (G), R4.2: now also U3.36 (ADC1_IN9/ADC2_IN9/TIM1_CH3N/TIM3_CH4/PB1); no longer U3.95 (CAN1_RX/I2C1_SCL/TIM4_CH3/PB8)
- net at Q3.1 (G), R3.2: now also U3.98 (PE1); no longer U3.96 (CAN1_TX/DAC_EXTI9/I2C1_SDA/TIM4_CH4/PB9)
- net at Q1.2 (D): now also J6.3 (Pin_3); no longer J6.7 (Pin_7)
- net at Q2.2 (D): now also J7.3 (Pin_3); no longer J7.7 (Pin_7)
- net at Q5.3 (D): now also J6.1 (Pin_1); no longer J6.5 (Pin_5)
- net at Q4.3 (D): now also J7.1 (Pin_1); no longer J7.5 (Pin_5)
- net at A1.3 (1B): now also J6.5 (Pin_5); no longer J6.1 (Pin_1)
- net at A1.4 (1A): now also J6.6 (Pin_6); no longer J6.2 (Pin_2)
- net at A1.5 (2A): now also J6.7 (Pin_7); no longer J6.3 (Pin_3)
- net at A1.6 (2B): now also J6.8 (Pin_8); no longer J6.4 (Pin_4)
- net at A2.3 (1B): now also J7.5 (Pin_5); no longer J7.1 (Pin_1)
- net at A2.4 (1A): now also J7.6 (Pin_6); no longer J7.2 (Pin_2)
- net at A2.5 (2A): now also J7.7 (Pin_7); no longer J7.3 (Pin_3)
- net at A2.6 (2B): now also J7.8 (Pin_8); no longer J7.4 (Pin_4)
- new net: LS1.1, U3.97 (PE0/TIM4_ETR)
- now unconnected: U3.72 (SYS_JTMS-SWDIO/PA13)
- no-connect marks 37 -> 38
Other:
- moved on the sheet: D3, D4, LS1

Commit message: Новая версия
Parts:
- removed C11, C12, C13, C14: 100nF, Capacitor_SMD:C_1206_3216Metric, symbol V2-rescue:C-device
- removed J31: Bed level, Connector_PinHeader_2.54mm:PinHeader_1x03_P2.54mm_Vertical_SMD_Pin1Left, symbol V2-rescue:Conn_01x03_Male-Connector
- added SW1: Bed Level nozle, Connector_JST:JST_EH_B02B-EH-A_1x02_P2.50mm_Vertical, symbol V2-rescue:SW_Push_Open-Switch
- added SW12: Bed Level, Connector_JST:JST_EH_B02B-EH-A_1x02_P2.50mm_Vertical, symbol V2-rescue:SW_Push_Open-Switch
Connections:
- net GNDD: now also SW1.2 (B), SW12.2 (B)
- net at U3.16 (ADC1_IN11/ADC2_IN11/PC1): now also SW12.1 (A)
- net at U3.9 (ADC1_EXTI15/ADC2_EXTI15/RCC_OSC32_OUT/PC15): now also SW1.1 (A)
- no-connect marks 38 -> 37
Changed lines of the file:
@@
 EESchema Schematic File Version 4
 LIBS:V2-cache
-EELAYER 26 0
+EELAYER 29 0
 EELAYER END
 $Descr A2 23386 16535
@@
 $EndComp
 $Comp
-L V2-rescue:GNDD-power #PWR0130
-U 1 1 5C497D89
-P 8050 15550
-F 0 "#PWR0130" H 8050 15300 50  0001 C CNN
-F 1 "GNDD" H 8054 15395 50  0000 C CNN
-F 2 "" H 8050 15550 50  0001 C CNN
-F 3 "" H 8050 15550 50  0001 C CNN
-	1    8050 15550
-	-1   0    0    1
-$EndComp
-$Comp
 L V2-rescue:GNDD-power #PWR0131
 U 1 1 5C4985EB
@@
 	0    1    1    0
 $EndComp
-$Comp
-L V2-rescue:C-device C8
-U 1 1 5D0DBFC1
-P 9800 5950
-F 0 "C8" H 9915 5996 50  0000 L CNN
-F 1 "4.7uF" H 9915 5905 50  0000 L CNN
-F 2 "Capacitor_SMD:C_1206_3216Metric" H 9838 5800 50  0001 C CNN
-F 3 "" H 9800 5950 50  0001 C CNN
-	1    9800 5950
-	1    0    0    -1
-$EndComp
-$Comp
-L V2-rescue:GNDD-power #PWR0220
-U 1 1 5D0DC263
-P 9800 5800
-F 0 "#PWR0220" H 9800 5550 50  0001 C CNN
-F 1 "GNDD" H 9804 5645 50  0000 C CNN
-F 2 "" H 9800 5800 50  0001 C CNN
-F 3 "" H 9800 5800 50  0001 C CNN
-	1    9800 5800
-	-1   0    0    1
-$EndComp
-Wire Wire Line
-	10600 6700 10600 6400
-$Comp
-L V2-rescue:C-device C10
-U 1 1 5D18CD97
-P 10250 5950
-F 0 "C10" H 10365 5996 50  0000 L CNN
-F 1 "100nF" H 10365 5905 50  0000 L CNN
-F 2 "Capacitor_SMD:C_1206_3216Metric" H 10288 5800 50  0001 C CNN
-F 3 "" H 10250 5950 50  0001 C CNN
-	1    10250 5950
-	1    0    0    -1
-$EndComp
-$Comp
-L V2-rescue:C-device C11
-U 1 1 5D1B9492
-P 10700 5950
-F 0 "C11" H 10815 5996 50  0000 L CNN
-F 1 "100nF" H 10815 5905 50  0000 L CNN
-F 2 "Capacitor_SMD:C_1206_3216Metric" H 10738 5800 50  0001 C CNN
-F 3 "" H 10700 5950 50  0001 C CNN
-	1    10700 5950
-	1    0    0    -1
-$EndComp
-$Comp
-L V2-rescue:C-device C12
-U 1 1 5D1B9544
-P 11150 5950
-F 0 "C12" H 11265 5996 50  0000 L CNN
-F 1 "100nF" H 11265 5905 50  0000 L CNN
-F 2 "Capacitor_SMD:C_1206_3216Metric" H 11188 5800 50  0001 C CNN
-F 3 "" H 11150 5950 50  0001 C CNN
-	1    11150 5950
-	1    0    0    -1
-$EndComp
-$Comp
-L V2-rescue:C-device C13
-U 1 1 5D1B95F6
-P 11600 5950
-F 0 "C13" H 11715 5996 50  0000 L CNN
-F 1 "100nF" H 11715 5905 50  0000 L CNN
-F 2 "Capacitor_SMD:C_1206_3216Metric" H 11638 5800 50  0001 C CNN
-F 3 "" H 11600 5950 50  0001 C CNN
-	1    11600 5950
-	1    0    0    -1
-$EndComp
-$Comp
-L V2-rescue:C-device C14
-U 1 1 5D1B96B0
-P 12050 5950
-F 0 "C14" H 12165 5996 50  0000 L CNN
-F 1 "100nF" H 12165 5905 50  0000 L CNN
-F 2 "Capacitor_SMD:C_1206_3216Metric" H 12088 5800 50  0001 C CNN
-F 3 "" H 12050 5950 50  0001 C CNN
-	1    12050 5950
-	1    0    0    -1
-$EndComp
-Wire Wire Line
-	10600 6400 10250 6400
-Wire Wire Line
-	10250 6400 10250 6100
-Wire Wire Line
-	10700 6700 10700 6100
-Wire Wire Line
-	10800 6700 10800 6150
-Wire Wire Line
-	10800 6150 11150 6150
-Wire Wire Line
-	11150 6150 11150 6100
-Wire Wire Line
-	10900 6700 10900 6200
-Wire Wire Line
-	10900 6200 11600 6200
-Wire Wire Line
-	11600 6200 11600 6100
-Wire Wire Line
-	11000 6250 12050 6250
-Wire Wire Line
-	12050 6250 12050 6100
-Wire Wire Line
-	10600 6700 10700 6700
-Connection ~ 10600 6700
-Connection ~ 10700 6700
-Wire Wire Line
-	10700 6700 10800 6700
-Connection ~ 10800 6700
-Wire Wire Line
-	10800 6700 10900 6700
-Connection ~ 10900 6700
-Wire Wire Line
-	10900 6700 11000 6700
-Wire Wire Line
-	11000 6250 11000 6700
-Connection ~ 11000 6700
-Wire Wire Line
-	11000 6700 11100 6700
-Connection ~ 11100 6700
-Wire Wire Line
-	10600 6700 9800 6700
-Wire Wire Line
-	9800 6700 9800 6100
-$Comp
-L V2-rescue:GNDD-power #PWR0221
-U 1 1 5D4196BD
-P 10250 5800
-F 0 "#PWR0221" H 10250 5550 50  0001 C CNN
-F 1 "GNDD" H 10254 5645 50  0000 C CNN
-F 2 "" H 10250 5800 50  0001 C CNN
-F 3 "" H 10250 5800 50  0001 C CNN
-	1    10250 5800
-	-1   0    0    1
-$EndComp
-$Comp
-L V2-rescue:GNDD-power #PWR0222
-U 1 1 5D419762
-P 10700 5800
-F 0 "#PWR0222" H 10700 5550 50  0001 C CNN
-F 1 "GNDD" H 10704 5645 50  0000 C CNN
-F 2 "" H 10700 5800 50  0001 C CNN
-F 3 "" H 10700 5800 50  0001 C CNN
-	1    10700 5800
-	-1   0    0    1
-$EndComp
-$Comp
-L V2-rescue:GNDD-power #PWR0223
-U 1 1 5D419807
-P 11150 5800
-F 0 "#PWR0223" H 11150 5550 50  0001 C CNN
-F 1 "GNDD" H 11154 5645 50  0000 C CNN
-F 2 "" H 11150 5800 50  0001 C CNN
-F 3 "" H 11150 5800 50  0001 C CNN
-	1    11150 5800
-	-1   0    0    1
-$EndComp
-$Comp
-L V2-rescue:GNDD-power #PWR0224
-U 1 1 5D4198AC
-P 11600 5800
-F 0 "#PWR0224" H 11600 5550 50  0001 C CNN
-F 1 "GNDD" H 11604 5645 50  0000 C CNN
-F 2 "" H 11600 5800 50  0001 C CNN
-F 3 "" H 11600 5800 50  0001 C CNN
-	1    11600 5800
-	-1   0    0    1
-$EndComp
-$Comp
-L V2-rescue:GNDD-power #PWR0225
-U 1 1 5D419951
-P 12050 5800
-F 0 "#PWR0225" H 12050 5550 50  0001 C CNN
-F 1 "GNDD" H 12054 5645 50  0000 C CNN
-F 2 "" H 12050 5800 50  0001 C CNN
-F 3 "" H 12050 5800 50  0001 C CNN
-	1    12050 5800
-	-1   0    0    1
-$EndComp
 Wire Wire Line
 	10600 12600 10700 12600
@@
 	7350 7400 8400 7400
 NoConn ~ 8400 7200
-NoConn ~ 13400 12100
 Wire Wire Line
 	4300 4550 4300 4500
@@
 $EndComp
 $Comp
-L V2-rescue:Conn_01x03_Male-Connector J31
-U 1 1 5C6206CB
-P 8150 15750
-F 0 "J31" V 8000 15750 50  0000 R CNN
-F 1 "Bed level" V 8100 15900 50  0000 R CNN
-F 2 "Connector_PinHeader_2.54mm:PinHeader_1x03_P2.54mm_Vertical_SMD_Pin1Left" H 8150 15750 50  0001 C CNN
-F 3 "~" H 8150 15750 50  0001 C CNN
-	1    8150 15750
-	0    -1   -1   0
-$EndComp
-$Comp
-L V2-rescue:+3.3V-power #PWR0241
-U 1 1 5C789638
-P 8250 15550
-F 0 "#PWR0241" H 8250 15400 50  0001 C CNN
-F 1 "+3.3V" H 8265 15723 50  0000 C CNN
-F 2 "" H 8250 15550 50  0001 C CNN
-F 3 "" H 8250 15550 50  0001 C CNN
-	1    8250 15550
-	1    0    0    -1
-$EndComp
-$Comp
 L POWER_LIB:PWR_FLAG #FLG0101
 U 1 1 5C534BEB
@@
 	14950 14800 8150 14800
 Wire Wire Line
-	8150 14800 8150 15550
-Wire Wire Line
 	8700 15350 8700 14750
 Wire Wire Line
@@
 Wire Wire Line
 	14650 7500 13400 7500
+$Comp
+L V2-rescue:GNDD-power #PWR0130
+U 1 1 5C497D89
+P 8150 15750
+F 0 "#PWR0130" H 8150 15500 50  0001 C CNN
+F 1 "GNDD" H 8154 15595 50  0000 C CNN
+F 2 "" H 8150 15750 50  0001 C CNN
+F 3 "" H 8150 15750 50  0001 C CNN
+	1    8150 15750
+	1    0    0    -1
+$EndComp
+$Comp
+L V2-rescue:SW_Push_Open-Switch SW12
+U 1 1 5CFCCBD5
+P 8150 15550
+F 0 "SW12" V 8104 15628 50  0000 L CNN
+F 1 "Bed Level" V 8195 15628 50  0000 L CNN
+F 2 "Connector_JST:JST_EH_B02B-EH-A_1x02_P2.50mm_Vertical" H 8150 15750 50  0001 C CNN
+F 3 "" H 8150 15750 50  0001 C CNN
+	1    8150 15550
+	0    1    1    0
+$EndComp
+Wire Wire Line
+	8150 14800 8150 15350
+$Comp
+L V2-rescue:SW_Push_Open-Switch SW1
+U 1 1 5D0AFB29
+P 7250 15550
+F 0 "SW1" V 7204 15628 50  0000 L CNN
+F 1 "Bed Level nozle" V 7295 15628 50  0000 L CNN
+F 2 "Connector_JST:JST_EH_B02B-EH-A_1x02_P2.50mm_Vertical" H 7250 15750 50  0001 C CNN
+F 3 "" H 7250 15750 50  0001 C CNN
+	1    7250 15550
+	0    1    1    0
+$EndComp
+$Comp
+L V2-rescue:GNDD-power #PWR0114
+U 1 1 5D0B183C
+P 7250 15750
+F 0 "#PWR0114" H 7250 15500 50  0001 C CNN
+F 1 "GNDD" H 7254 15595 50  0000 C CNN
+F 2 "" H 7250 15750 50  0001 C CNN
+F 3 "" H 7250 15750 50  0001 C CNN
+	1    7250 15750
+	1    0    0    -1
+$EndComp
+Wire Wire Line
+	13400 12100 14600 12100
+Wire Wire Line
+	14600 12100 14600 14900
+Wire Wire Line
+	14600 14900 7250 14900
+Wire Wire Line
+	7250 14900 7250 15350
+Connection ~ 11100 6700
+Wire Wire Line
+	11000 6700 11100 6700
+Connection ~ 11000 6700
+Wire Wire Line
+	10900 6700 11000 6700
+Connection ~ 10900 6700
+Wire Wire Line
+	10800 6700 10900 6700
+Connection ~ 10800 6700
+Wire Wire Line
+	10700 6700 10800 6700
+Connection ~ 10700 6700
+Wire Wire Line
+	10600 6700 10700 6700
+Connection ~ 10600 6700
+Wire Wire Line
+	10600 6700 9800 6700
+Wire Wire Line
+	10600 6700 10600 6400
+Wire Wire Line
+	10600 6400 10250 6400
+Wire Wire Line
+	9800 6700 9800 6100
+Wire Wire Line
+	10250 6400 10250 6100
+$Comp
+L V2-rescue:C-device C10
+U 1 1 5D18CD97
+P 10250 5950
+F 0 "C10" H 10365 5996 50  0000 L CNN
+F 1 "100nF" H 10365 5905 50  0000 L CNN
+F 2 "Capacitor_SMD:C_1206_3216Metric" H 10288 5800 50  0001 C CNN
+F 3 "" H 10250 5950 50  0001 C CNN
+	1    10250 5950
+	1    0    0    -1
+$EndComp
+$Comp
+L V2-rescue:GNDD-power #PWR0221
+U 1 1 5D4196BD
+P 10250 5800
+F 0 "#PWR0221" H 10250 5550 50  0001 C CNN
+F 1 "GNDD" H 10254 5645 50  0000 C CNN
+F 2 "" H 10250 5800 50  0001 C CNN
+F 3 "" H 10250 5800 50  0001 C CNN
+	1    10250 5800
+	-1   0    0    1
+$EndComp
+$Comp
+L V2-rescue:GNDD-power #PWR0220
+U 1 1 5D0DC263
+P 9800 5800
+F 0 "#PWR0220" H 9800 5550 50  0001 C CNN
+F 1 "GNDD" H 9804 5645 50  0000 C CNN
+F 2 "" H 9800 5800 50  0001 C CNN
+F 3 "" H 9800 5800 50  0001 C CNN
+	1    9800 5800
+	-1   0    0    1
+$EndComp
+$Comp
+L V2-rescue:C-device C8
+U 1 1 5D0DBFC1
+P 9800 5950
+F 0 "C8" H 9915 5996 50  0000 L CNN
+F 1 "4.7uF" H 9915 5905 50  0000 L CNN
+F 2 "Capacitor_SMD:C_1206_3216Metric" H 9838 5800 50  0001 C CNN
+F 3 "" H 9800 5950 50  0001 C CNN
+	1    9800 5950
+	1    0    0    -1
+$EndComp
 $EndSCHEMATC

Commit message: переразвёл заново
Parts:
- 47uH1: footprint Inductor_SMD:L_1206_3216Metric -> Inductor_THT:L_Radial_D12.0mm_P6.00mm_MuRATA_1900R
- C1: footprint Capacitor_SMD:CP_Elec_10x10.5 -> Capacitor_THT:CP_Radial_D10.0mm_P5.00mm
- C2: footprint Capacitor_SMD:CP_Elec_10x10.5 -> Capacitor_THT:CP_Radial_D10.0mm_P7.50mm
- D1: footprint Diode_SMD:D_2512_6332Metric_Castellated -> Diode_SMD:SS14
- D2: footprint w_smd_diode:do214ac -> w_smd_diode:do214ab
- J1, J3: footprint TerminalBlock_4Ucon:TerminalBlock_4Ucon_1x02_P3.50mm_Horizontal -> TerminalBlock_RND:TerminalBlock_RND_205-00045_1x02_P5.00mm_Horizontal
- Q1, Q2: footprint Package_TO_SOT_SMD:SOT-223-3_TabPin2 -> Package_TO_SOT_SMD:TO-252-2
- Q3, Q4, Q5, Q6: footprint Package_TO_SOT_SMD:TO-252-3_TabPin2 -> Package_TO_SOT_SMD:TO-252-2
- U2: footprint Package_TO_SOT_SMD:TO-252-3_TabPin2 -> Package_TO_SOT_SMD:SOT-223-3_TabPin2
Connections:
- net +3V3: now also U2.2 (GND); no longer U2.3 (OUT)
- net +5VD: now also U2.3 (OUT); no longer U2.1 (IN)
- net GNDD: now also U2.1 (IN); no longer U2.2 (GND)
Changed lines of the file:
@@
 L V2-rescue:GNDD-power #PWR0101
 U 1 1 5C43815D
-P 4450 1400
-F 0 "#PWR0101" H 4450 1150 50  0001 C CNN
-F 1 "GNDD" H 4454 1245 50  0000 C CNN
-F 2 "" H 4450 1400 50  0001 C CNN
-F 3 "" H 4450 1400 50  0001 C CNN
-	1    4450 1400
-	1    0    0    -1
+P 4150 1100
+F 0 "#PWR0101" H 4150 850 50  0001 C CNN
+F 1 "GNDD" H 4154 945 50  0000 C CNN
+F 2 "" H 4150 1100 50  0001 C CNN
+F 3 "" H 4150 1100 50  0001 C CNN
+	1    4150 1100
+	0    1    1    0
 $EndComp
 $Comp
@@
 F 0 "D1" V 2500 1650 50  0000 L CNN
 F 1 "SS54" V 2600 1650 50  0000 L CNN
-F 2 "Diode_SMD:D_2512_6332Metric_Castellated" H 2500 1425 50  0001 C CNN
+F 2 "Diode_SMD:SS14" H 2500 1425 50  0001 C CNN
 F 3 "http://www.vishay.com/docs/88526/1n5820.pdf" H 2500 1600 50  0001 C CNN
 	1    2500 1600
@@
 F 0 "47uH1" V 2700 1450 50  0000 C CNN
 F 1 "L?" V 2849 1450 50  0000 C CNN
-F 2 "Inductor_SMD:L_1206_3216Metric" H 2750 1450 50  0001 C CNN
+F 2 "Inductor_THT:L_Radial_D12.0mm_P6.00mm_MuRATA_1900R" H 2750 1450 50  0001 C CNN
 F 3 "" H 2750 1450 50  0001 C CNN
 	1    2750 1450
@@
 F 0 "C1" H 1132 954 50  0000 R CNN
 F 1 "680uF" H 1132 1045 50  0000 R CNN
-F 2 "Capacitor_SMD:CP_Elec_10x10.5" H 1288 850 50  0001 C CNN
+F 2 "Capacitor_THT:CP_Radial_D10.0mm_P5.00mm" H 1288 850 50  0001 C CNN
 F 3 "" H 1250 1000 50  0001 C CNN
 	1    1250 1000
@@
 F 0 "C2" H 3118 1646 50  0000 L CNN
 F 1 "220uF" H 3118 1555 50  0000 L CNN
-F 2 "Capacitor_SMD:CP_Elec_10x10.5" H 3038 1450 50  0001 C CNN
+F 2 "Capacitor_THT:CP_Radial_D10.0mm_P7.50mm" H 3038 1450 50  0001 C CNN
 F 3 "" H 3000 1600 50  0001 C CNN
 	1    3000 1600
@@
 L V2-rescue:+5VD-power #PWR0111
 U 1 1 5C44D470
-P 4150 1100
-F 0 "#PWR0111" H 4150 950 50  0001 C CNN
-F 1 "+5VD" V 4165 1228 50  0000 L CNN
-F 2 "" H 4150 1100 50  0001 C CNN
-F 3 "" H 4150 1100 50  0001 C CNN
-	1    4150 1100
-	0    -1   -1   0
+P 4750 1100
+F 0 "#PWR0111" H 4750 950 50  0001 C CNN
+F 1 "+5VD" V 4765 1228 50  0000 L CNN
+F 2 "" H 4750 1100 50  0001 C CNN
+F 3 "" H 4750 1100 50  0001 C CNN
+	1    4750 1100
+	0    1    1    0
 $EndComp
 $Comp
@@
 F 0 "D2" H 7400 834 50  0000 C CNN
 F 1 "1n5819" H 7400 925 50  0000 C CNN
-F 2 "w_smd_diode:do214ac" H 7400 1050 50  0001 C CNN
+F 2 "w_smd_diode:do214ab" H 7400 1050 50  0001 C CNN
 F 3 "" H 7400 1050 50  0001 C CNN
 	1    7400 1050
@@
 F 0 "U2" H 4450 1342 50  0000 C CNN
 F 1 "R-783.3-1.0" H 4450 1251 50  0000 C CNN
-F 2 "Package_TO_SOT_SMD:TO-252-3_TabPin2" H 4500 850 50  0001 L CIN
+F 2 "Package_TO_SOT_SMD:SOT-223-3_TabPin2" H 4500 850 50  0001 L CIN
 F 3 "https://www.recom-power.com/pdf/Innoline/R-78xx-1.0.pdf" H 4450 1100 50  0001 C CNN
 	1    4450 1100
@@
 L V2-rescue:+3.3V-power #PWR0118
 U 1 1 5C45FD0D
-P 4750 1100
-F 0 "#PWR0118" H 4750 950 50  0001 C CNN
-F 1 "+3.3V" V 4765 1228 50  0000 L CNN
-F 2 "" H 4750 1100 50  0001 C CNN
-F 3 "" H 4750 1100 50  0001 C CNN
-	1    4750 1100
-	0    1    1    0
+P 4450 1400
+F 0 "#PWR0118" H 4450 1250 50  0001 C CNN
+F 1 "+3.3V" V 4465 1528 50  0000 L CNN
+F 2 "" H 4450 1400 50  0001 C CNN
+F 3 "" H 4450 1400 50  0001 C CNN
+	1    4450 1400
+	-1   0    0    1
 $EndComp
 $Comp
@@
 F 0 "Q1" H 1006 4796 50  0000 L CNN
 F 1 "STN4NF20L" H 1006 4705 50  0000 L CNN
-F 2 "Package_TO_SOT_SMD:SOT-223-3_TabPin2" H 1000 4675 50  0001 L CIN
+F 2 "Package_TO_SOT_SMD:TO-252-2" H 1000 4675 50  0001 L CIN
 F 3 "https://www.infineon.com/dgdl/Infineon-BSP129-DS-v01_42-en.pdf?fileId=db3a30433c1a8752013c1fc296d2395f" H 800 4750 50  0001 L CNN
 	1    800  4750
@@
 F 0 "Q2" H 1906 4796 50  0000 L CNN
 F 1 "STN4NF20L" H 1906 4705 50  0000 L CNN
-F 2 "Package_TO_SOT_SMD:SOT-223-3_TabPin2" H 1900 4675 50  0001 L CIN
+F 2 "Package_TO_SOT_SMD:TO-252-2" H 1900 4675 50  0001 L CIN
 F 3 "https://www.infineon.com/dgdl/Infineon-BSP129-DS-v01_42-en.pdf?fileId=db3a30433c1a8752013c1fc296d2395f" H 1700 4750 50  0001 L CNN
 	1    1700 4750
@@
 F 0 "J3" V 2710 4241 50  0000 L CNN
 F 1 "Bed Heater" V 2550 3950 50  0000 L CNN
-F 2 "TerminalBlock_4Ucon:TerminalBlock_4Ucon_1x02_P3.50mm_Horizontal" H 2650 4200 50  0001 C CNN
+F 2 "TerminalBlock_RND:TerminalBlock_RND_205-00045_1x02_P5.00mm_Horizontal" H 2650 4200 50  0001 C CNN
 F 3 "~" H 2650 4200 50  0001 C CNN
 	1    2650 4200
@@
 F 0 "Q4" H 3550 4800 50  0000 L CNN
 F 1 "04N03LA" H 3550 4700 50  0000 L CNN
-F 2 "Package_TO_SOT_SMD:TO-252-3_TabPin2" H 3550 4675 50  0001 L CIN
+F 2 "Package_TO_SOT_SMD:TO-252-2" H 3550 4675 50  0001 L CIN
 F 3 "https://www.fairchildsemi.com/datasheets/BS/BSS138.pdf" H 3350 4750 50  0001 L CNN
 	1    3350 4750
@@
 F 0 "Q3" H 2750 4800 50  0000 L CNN
 F 1 "04N03LA" H 2750 4700 50  0000 L CNN
-F 2 "Package_TO_SOT_SMD:TO-252-3_TabPin2" H 2750 4675 50  0001 L CIN
+F 2 "Package_TO_SOT_SMD:TO-252-2" H 2750 4675 50  0001 L CIN
 F 3 "https://www.fairchildsemi.com/datasheets/BS/BSS138.pdf" H 2550 4750 50  0001 L CNN
 	1    2550 4750
@@
 F 0 "Q5" H 4400 4800 50  0000 L CNN
 F 1 "04N03LA" H 4400 4700 50  0000 L CNN
-F 2 "Package_TO_SOT_SMD:TO-252-3_TabPin2" H 4400 4675 50  0001 L CIN
+F 2 "Package_TO_SOT_SMD:TO-252-2" H 4400 4675 50  0001 L CIN
 F 3 "https://www.fairchildsemi.com/datasheets/BS/BSS138.pdf" H 4200 4750 50  0001 L CNN
 	1    4200 4750
@@
 F 0 "Q6" H 20750 10550 50  0000 L CNN
 F 1 "04N03LA" H 20750 10450 50  0000 L CNN
-F 2 "Package_TO_SOT_SMD:TO-252-3_TabPin2" H 20750 10425 50  0001 L CIN
+F 2 "Package_TO_SOT_SMD:TO-252-2" H 20750 10425 50  0001 L CIN
 F 3 "https://www.fairchildsemi.com/datasheets/BS/BSS138.pdf" H 20550 10500 50  0001 L CNN
 	1    20550 10500
@@
 F 0 "J1" V 10973 1180 50  0000 L CNN
 F 1 "Input voltage" V 11064 1180 50  0000 L CNN
-F 2 "TerminalBlock_4Ucon:TerminalBlock_4Ucon_1x02_P3.50mm_Horizontal" H 11100 1100 50  0001 C CNN
+F 2 "TerminalBlock_RND:TerminalBlock_RND_205-00045_1x02_P5.00mm_Horizontal" H 11100 1100 50  0001 C CNN
 F 3 "~" H 11100 1100 50  0001 C CNN
 	1    11100 1100
